File: leds-smd.sch (EAGLE design)
At the start: 66 parts

Commit message: Added support for 5mm leds
Parts:
- R1, R10, R11, R12, R13, R14, R15, R16, R2, R3, R4, R5, R6, R7, R8, R9: value 150 -> 120
Other:
- note added: "12V"
Changed lines of the file:
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@@
 </classes>
 <parts>
-<part name="R1" library="resistor" deviceset="R-EU_" device="M1206" value="150"/>
+<part name="R1" library="resistor" deviceset="R-EU_" device="M1206" value="120"/>
 <part name="LD1" library="adafruit" deviceset="LED" device="5MM"/>
 <part name="LD4" library="adafruit" deviceset="LED" device="5MM"/>
@@
 <part name="LD16" library="adafruit" deviceset="LED" device="5MM"/>
 <part name="LD19" library="adafruit" deviceset="LED" device="5MM"/>
-<part name="R2" library="resistor" deviceset="R-EU_" device="M1206" value="150"/>
-<part name="R3" library="resistor" deviceset="R-EU_" device="M1206" value="150"/>
-<part name="R4" library="resistor" deviceset="R-EU_" device="M1206" value="150"/>
-<part name="R5" library="resistor" deviceset="R-EU_" device="M1206" value="150"/>
-<part name="R6" library="resistor" deviceset="R-EU_" device="M1206" value="150"/>
-<part name="R7" library="resistor" deviceset="R-EU_" device="M1206" value="150"/>
+<part name="R2" library="resistor" deviceset="R-EU_" device="M1206" value="120"/>
+<part name="R3" library="resistor" deviceset="R-EU_" device="M1206" value="120"/>
+<part name="R4" library="resistor" deviceset="R-EU_" device="M1206" value="120"/>
+<part name="R5" library="resistor" deviceset="R-EU_" device="M1206" value="120"/>
+<part name="R6" library="resistor" deviceset="R-EU_" device="M1206" value="120"/>
+<part name="R7" library="resistor" deviceset="R-EU_" device="M1206" value="120"/>
 <part name="LD2" library="adafruit" deviceset="LED" device="5MM"/>
 <part name="LD3" library="adafruit" deviceset="LED" device="5MM"/>
@@
 <part name="LD20" library="adafruit" deviceset="LED" device="5MM"/>
 <part name="LD21" library="adafruit" deviceset="LED" device="5MM"/>
-<part name="R8" library="resistor" deviceset="R-EU_" device="M1206" value="150"/>
-<part name="R9" library="resistor" deviceset="R-EU_" device="M1206" value="150"/>
-<part name="R10" library="resistor" deviceset="R-EU_" device="M1206" value="150"/>
-<part name="R11" library="resistor" deviceset="R-EU_" device="M1206" value="150"/>
-<part name="R12" library="resistor" deviceset="R-EU_" device="M1206" value="150"/>
-<part name="R13" library="resistor" deviceset="R-EU_" device="M1206" value="150"/>
-<part name="R14" library="resistor" deviceset="R-EU_" device="M1206" value="150"/>
+<part name="R8" library="resistor" deviceset="R-EU_" device="M1206" value="120"/>
+<part name="R9" library="resistor" deviceset="R-EU_" device="M1206" value="120"/>
+<part name="R10" library="resistor" deviceset="R-EU_" device="M1206" value="120"/>
+<part name="R11" library="resistor" deviceset="R-EU_" device="M1206" value="120"/>
+<part name="R12" library="resistor" deviceset="R-EU_" device="M1206" value="120"/>
+<part name="R13" library="resistor" deviceset="R-EU_" device="M1206" value="120"/>
+<part name="R14" library="resistor" deviceset="R-EU_" device="M1206" value="120"/>
 <part name="LD22" library="adafruit" deviceset="LED" device="5MM"/>
 <part name="LD25" library="adafruit" deviceset="LED" device="5MM"/>
@@
 <part name="LD42" library="adafruit" deviceset="LED" device="5MM"/>
 <part name="SV2" library="con-lstb" deviceset="MA03-1" device=""/>
-<part name="R15" library="resistor" deviceset="R-EU_" device="M1206" value="150"/>
+<part name="R15" library="resistor" deviceset="R-EU_" device="M1206" value="120"/>
 <part name="LD43" library="adafruit" deviceset="LED" device="5MM"/>
 <part name="LD44" library="adafruit" deviceset="LED" device="5MM"/>
 <part name="LD45" library="adafruit" deviceset="LED" device="5MM"/>
-<part name="R16" library="resistor" deviceset="R-EU_" device="M1206" value="150"/>
+<part name="R16" library="resistor" deviceset="R-EU_" device="M1206" value="120"/>
 <part name="LD46" library="adafruit" deviceset="LED" device="5MM"/>
 <part name="LD47" library="adafruit" deviceset="LED" device="5MM"/>
@@
 <part name="SUPPLY2" library="supply2" deviceset="GND" device=""/>
 <part name="SUPPLY3" library="supply2" deviceset="GND" device=""/>
+<part name="FRAME1" library="frames" deviceset="DINA4_L" device=""/>
 </parts>
 <sheets>
 <sheet>
 <plain>
+<text x="-33.02" y="104.14" size="1.778" layer="96">12V</text>
 </plain>
 <instances>
@@
 <instance part="SUPPLY2" gate="GND" x="22.86" y="2.54"/>
 <instance part="SUPPLY3" gate="GND" x="99.06" y="2.54"/>
+<instance part="FRAME1" gate="G$1" x="-96.52" y="-50.8"/>
+<instance part="FRAME1" gate="G$2" x="66.04" y="-50.8"/>
 </instances>
 <busses>
